File: PCB_Main2/PCB_Main2.kicad_sch (KiCad schematic)
At the start: 0 parts

Commit message: update PCB_Main1 & PCB_Main2
Parts:
- added D1: D, symbol Device:D
- added J1: GPS, symbol Connector:Conn_01x05_Female
- added J2: Micro_SD_Card_Det_Hirose_DM3AT, symbol Connector:Micro_SD_Card_Det_Hirose_DM3AT
- added JP1: SolderJumper_2_Open, symbol Jumper:SolderJumper_2_Open
- added U1: MOUDLE-SEEEDUINO-XIAO, symbol MOUDLE-SEEEDUINO-XIAO:MOUDLE-SEEEDUINO-XIAO
- added U2: TWE-L-DP-W, Package_DIP:DIP-28_W15.24mm, symbol RF_ZigBee:TWE-L-DP-W
- added XH1: TWELITE_GPS_UART, symbol Connector:Conn_01x05_Female
- added XH2: SD-UART, symbol Connector:Conn_01x04_Female
Connections:
- new net: JP1.2 (B), U2.13 (DIO10/M1)
- new net: D1.1 (K), U1.14 (5V)
- new net +3V3: U2.28 (VCC), XH2.2 (Pin_2)
- new net +5V: D1.2 (A), J1.2 (Pin_2), XH1.2 (Pin_2)
- new net 1GPS: J1.5 (Pin_5), XH1.5 (Pin_5)
- new net GND: J1.1 (Pin_1), J2.6 (VSS), JP1.1 (A), U1.13 (GND), U2.1 (GND), U2.14 (GND), XH1.1 (Pin_1), XH2.1 (Pin_1)
- new net L_SD: U1.2 (PA4_A1_D1), XH2.4 (Pin_4)
- new net P3V3: J2.4 (VDD), U1.12 (3V3)
- new net PRGT: J1.4 (Pin_4), XH1.4 (Pin_4)
- new net PTSR: U1.8 (PB09_A7_D7_RX), U2.3 (DIO7/RX), XH2.3 (Pin_3)
- new net PTTR: XH1.3 (Pin_3)
- new net SD-CLK: J2.5 (CLK), U1.9 (PA7_A8_D8_SCK)
- new net SD-CS: J2.2 (DAT3/CD), U1.1 (PA02_A0_D0)
- new net SD-MISO: J2.7 (DAT0), U1.10 (PA5_A9_D9_MISO)
- new net SD-MOSI: J2.3 (CMD), U1.11 (PA6_A10_D10_MOSI)
- no-connect marks 0 -> 33
Other:
- company: (none) -> TORICA-24th
- title: (none) -> Main_2

Commit message: update README.md
Connections:
- net PTSR: no longer U2.3 (DIO7/RX)
- net PTTR: now also U2.3 (DIO7/RX)
- no-connect marks 33 -> 32
Changed lines of the file:
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@@
   (no_connect (at 76.2 105.41))
   (no_connect (at 33.655 48.895))
-  (no_connect (at 163.83 79.375))
   (no_connect (at 76.2 102.87))
   (no_connect (at 33.655 31.115))
@@
     (effects (font (size 1.27 1.27)) (justify left bottom))
   )
-  (label "PTSR" (at 85.725 100.33 180) (fields_autoplaced)
+  (label "PTTR" (at 85.725 100.33 180) (fields_autoplaced)
     (effects (font (size 1.27 1.27)) (justify right bottom))
   )

Commit message: Update PCB_Main
Parts:
- D1: footprint (none) -> Diode_THT:D_A-405_P10.16mm_Horizontal
- J1, XH2: footprint (none) -> Connector_JST:JST_XH_S5B-XH-A_1x05_P2.50mm_Horizontal
- J2: footprint (none) -> microSD:microSD_AE-MICRO-SD-DIP
- JP1: footprint (none) -> Jumper:SolderJumper-2_P1.3mm_Open_RoundedPad1.0x1.5mm
- U1: footprint (none) -> XIAO_PCB:MOUDLE14P-2.54-21X17.8MM
- XH1: footprint (none) -> Connector_JST:JST_XH_S4B-XH-A_1x04_P2.50mm_Horizontal
Changed lines of the file:
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@@
       (effects (font (size 1.27 1.27)))
     )
-    (property "Footprint" "" (at 105.41 39.37 0)
+    (property "Footprint" "Connector_JST:JST_XH_S5B-XH-A_1x05_P2.50mm_Horizontal" (at 105.41 39.37 0)
       (effects (font (size 1.27 1.27)) hide)
     )
@@
       (effects (font (size 1.27 1.27)) (justify right))
     )
-    (property "Footprint" "" (at 163.195 72.39 0)
+    (property "Footprint" "Diode_THT:D_A-405_P10.16mm_Horizontal" (at 163.195 72.39 0)
       (effects (font (size 1.27 1.27)) hide)
     )
@@
       (effects (font (size 1.27 1.27)))
     )
-    (property "Footprint" "" (at 34.29 77.47 0)
+    (property "Footprint" "Jumper:SolderJumper-2_P1.3mm_Open_RoundedPad1.0x1.5mm" (at 34.29 77.47 0)
       (effects (font (size 1.27 1.27)) hide)
     )
@@
       (effects (font (size 1.27 1.27)))
     )
-    (property "Footprint" "" (at 158.115 49.53 0)
+    (property "Footprint" "Connector_JST:JST_XH_S5B-XH-A_1x05_P2.50mm_Horizontal" (at 158.115 49.53 0)
       (effects (font (size 1.27 1.27)) hide)
     )
@@
       (effects (font (size 1.27 1.27)))
     )
-    (property "Footprint" "" (at 108.585 23.495 0)
+    (property "Footprint" "microSD:microSD_AE-MICRO-SD-DIP" (at 108.585 23.495 0)
       (effects (font (size 1.27 1.27)) hide)
     )
@@
       (effects (font (size 1.27 1.27)))
     )
-    (property "Footprint" "" (at 158.115 29.21 0)
+    (property "Footprint" "Connector_JST:JST_XH_S4B-XH-A_1x04_P2.50mm_Horizontal" (at 158.115 29.21 0)
       (effects (font (size 1.27 1.27)) hide)
     )
@@
       (effects (font (size 1.27 1.27)))
     )
-    (property "Footprint" "" (at 118.11 82.55 0)
-      (effects (font (size 1.27 1.27)) hide)
-    )
+    (property "Footprint" "XIAO_PCB:MOUDLE14P-2.54-21X17.8MM" (at 118.11 82.55 0)
+      (effects (font (size 1.27 1.27)) hide)
+    )

Commit message: Update PCB_Main
Parts:
- XH1: footprint Connector_JST:JST_XH_S4B-XH-A_1x04_P2.50mm_Horizontal -> Connector_JST:JST_XH_S5B-XH-A_1x05_P2.50mm_Horizontal
- XH2: footprint Connector_JST:JST_XH_S5B-XH-A_1x05_P2.50mm_Horizontal -> Connector_JST:JST_XH_S4B-XH-A_1x04_P2.50mm_Horizontal
Changed lines of the file:
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@@
       (effects (font (size 1.27 1.27)))
     )
-    (property "Footprint" "Connector_JST:JST_XH_S5B-XH-A_1x05_P2.50mm_Horizontal" (at 158.115 49.53 0)
+    (property "Footprint" "Connector_JST:JST_XH_S4B-XH-A_1x04_P2.50mm_Horizontal" (at 158.115 49.53 0)
       (effects (font (size 1.27 1.27)) hide)
     )
@@
       (effects (font (size 1.27 1.27)))
     )
-    (property "Footprint" "Connector_JST:JST_XH_S4B-XH-A_1x04_P2.50mm_Horizontal" (at 158.115 29.21 0)
+    (property "Footprint" "Connector_JST:JST_XH_S5B-XH-A_1x05_P2.50mm_Horizontal" (at 158.115 29.21 0)
       (effects (font (size 1.27 1.27)) hide)
     )
