File: PCB_Main2/PCB_Main2.kicad_pcb (KiCad board)
At the start: 2 copper layers, 115 x 115 mm, 12 parts, among them J1 GPS, J2 Micro_SD_Card_Det_Hirose_DM3AT, U1 MOUDLE-SEEEDUINO-XIAO, U2 TWE-L-DP-W

Commit message: Update PCB_Main
Parts:
- moved J1 66.3 mm to (183.7, 135.4), turned to 90 degrees
- moved XH1 60.1 mm to (163.3, 72.3), turned to 180 degrees
- moved J2 21.0 mm to (124.7, 91.0), turned to -90 degrees
Routing:
- net /PTTR: track 95.2 -> 178.0 mm
- net GND: track 246.2 -> 321.3 mm
- net /SD-CLK: track 142.5 -> 71.1 mm
- net /SD-CS: track 138.2 -> 75.8 mm
- net /SD-MOSI: track 104.6 -> 73.6 mm, vias 4 -> 2
- net /P3V3: track 105.1 -> 81.8 mm, vias 4 -> 2
- net /1GPS: track 71.7 -> 81.3 mm, vias 2 -> 0
- net /SD-MISO: track 88.0 -> 80.1 mm, vias 4 -> 2
- net /PRGT: track 73.4 -> 80.8 mm
- net +5V: track 91.2 -> 85.9 mm
