File: PCB_Main2/PCB_Main2.kicad_pcb (KiCad board)
At the start: 2 copper layers, 115 x 115 mm, 12 parts, among them J1 GPS, J2 Micro_SD_Card_Det_Hirose_DM3AT, U1 MOUDLE-SEEEDUINO-XIAO, U2 TWE-L-DP-W

Commit message: Update PCB_Main
Parts:
- moved J1 46.9 mm to (136.8, 136.1)
- moved U2 4.35 mm to (106.7, 114.0)
Routing:
- net /PTTR: track 178.0 -> 89.0 mm, vias 2 -> 0
- net GND: track 321.3 -> 265.3 mm
- net +5V: track 85.9 -> 114.4 mm
- net /1GPS: track 81.3 -> 69.8 mm, vias 0 -> 2
- net Net-(JP1-B): track 39.4 -> 34.2 mm
- net +3V3: track 55.9 -> 59.0 mm, vias 0 -> 2
- net /PRGT: track 80.8 -> 77.9 mm
