File: PCB_Main1/PCB_Main1.kicad_pcb (KiCad board)
At the start: 2 copper layers, 33 parts, among them M78AR033-1 R-78E3.3-0.5, M78AR05-1 M78AR05, M78AR05-2 M78AR05, M78AR05-3 M78AR05, M78AR05-4 M78AR05, SW1 SW_ICS, U1 Pico, U2 AE-BNO055, U3 DPS310

Commit message: Update PCB_Main
Parts:
- added REF**: DHM3, Library:DHM3, F.Cu at (80.0, 157.5)
- added REF**: DHM3, Library:DHM3, F.Cu at (187.0, 157.5)
- added REF**: DHM3, Library:DHM3, F.Cu at (80.0, 50.5)
- added REF**: DHM3, Library:DHM3, F.Cu at (187.0, 50.5)
- moved U3 137.1 mm to (170.7, 96.1), turned to 90 degrees
- moved M78AR05-4 129.9 mm to (151.2, 86.4), turned to 180 degrees
- moved U2 127.8 mm to (151.4, 123.4)
- moved C1 109.9 mm to (146.9, 103.0)
- moved D15 93.7 mm to (152.1, 79.7), turned to 90 degrees
- moved SW1 92.0 mm to (88.8, 135.4)
- moved D2 47.7 mm to (86.3, 70.3), turned to -90 degrees
- moved D4 36.6 mm to (103.9, 70.5), turned to -90 degrees
- moved D6 32.9 mm to (92.2, 80.6), turned to 90 degrees
- moved D5 32.9 mm to (158.6, 145.5), turned to 0 degrees
- moved M78AR05-2 29.2 mm to (92.1, 86.2), turned to 180 degrees
- moved ICS-board1 27.2 mm to (162.4, 51.3)
- moved XH4 26.9 mm to (97.5, 98.6), turned to -90 degrees
- moved D16 26.5 mm to (145.6, 69.4), turned to -90 degrees
- moved XH2 23.1 mm to (97.5, 116.1), turned to -90 degrees
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Routing:
- net GND: track 96.2 -> 617.7 mm, vias 0 -> 8
- net /IRXT: track 0.00 -> 287.6 mm, vias 0 -> 4
- net VCC: track 0.00 -> 228.0 mm, vias 0 -> 8
- net /SCL: track 0.00 -> 177.4 mm, vias 0 -> 4
- net /1GPS: track 0.00 -> 172.7 mm, vias 0 -> 2
- net /SPK: track 0.00 -> 142.7 mm, vias 0 -> 2
- net /SDA: track 0.00 -> 134.5 mm, vias 0 -> 5
- net /PRAT: track 0.00 -> 130.5 mm, vias 0 -> 4
- net /PTAR: track 0.00 -> 119.1 mm, vias 0 -> 4
- net /L_Under: track 0.00 -> 117.1 mm, vias 0 -> 2
- net +5V: track 0.00 -> 110.1 mm, vias 0 -> 2
- net /ITXR: track 0.00 -> 108.3 mm, vias 0 -> 2
- net /EN: track 0.00 -> 107.4 mm, vias 0 -> 4
- net +3V3: track 0.00 -> 105.4 mm, vias 0 -> 2
- net /L_SD: track 0.00 -> 102.6 mm, vias 0 -> 2
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- added copper zone on B.Cu, net GND
- added copper zone on F.Cu, net GND
Other:
- board outline added: 115 x 115 mm

Commit message: Update PCB_Main
Parts:
- moved XH1 9.34 mm to (176.1, 144.8), turned to 90 degrees
- moved XH5 7.55 mm to (176.1, 125.1), turned to 90 degrees
- moved SW1 3.84 mm to (85.0, 134.9)
- moved D5 0.49 mm to (159.1, 145.4)
- moved D1 0.48 mm to (169.4, 139.7)
- moved U1 0.33 mm to (126.6, 127.2), turned to 180 degrees
Routing:
- net GND: track 617.7 -> 457.5 mm, vias 8 -> 10
- net /IRXT: track 287.6 -> 165.2 mm, vias 4 -> 6
- net Net-(SW1A-B): track 30.9 -> 128.8 mm, vias 2 -> 4
- net /SCL: track 177.4 -> 88.2 mm, vias 4 -> 2
- net /PRUT: track 22.0 -> 111.1 mm, vias 0 -> 2
- net /L_Under: track 117.1 -> 29.2 mm
- net /PTUR: track 22.0 -> 108.5 mm
- net /SPK: track 142.7 -> 57.8 mm
- net +3V3: track 105.4 -> 189.7 mm, vias 2 -> 6
- net /PRAT: track 130.5 -> 49.7 mm, vias 4 -> 2
- net +5V: track 110.1 -> 181.3 mm
- net /PTAR: track 119.1 -> 55.2 mm, vias 4 -> 2
- net /SDA: track 134.5 -> 78.6 mm, vias 5 -> 4
- net /L_ICS: track 100.0 -> 44.1 mm, vias 2 -> 4
- net /PTSR: track 100.7 -> 74.2 mm, vias 4 -> 2
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
Commit message: Update PCB_Main
Parts:
- moved D3 10.8 mm to (130.4, 80.7), turned to 90 degrees
- moved D7 9.84 mm to (125.2, 70.5), turned to -90 degrees
- moved D15 2.75 mm to (149.5, 80.6)
- moved D4 2.23 mm to (106.2, 70.5)
- moved M78AR05-3 1.98 mm to (111.3, 86.2)
- moved D8 1.97 mm to (111.3, 80.6)
- moved M78AR05-4 1.72 mm to (149.5, 86.2)
- moved D16 1.57 mm to (144.4, 70.4)
- moved M78AR033-1 1.27 mm to (130.4, 86.2)
- moved D2 0.74 mm to (87.0, 70.4)
Routing:
- net GND: track 457.5 -> 240.1 mm, vias 10 -> 2
- net +5V: track 181.3 -> 210.2 mm, vias 2 -> 4
- net Net-(D3-K): track 6.42 -> 25.2 mm, vias 0 -> 2
- net VCC: track 245.6 -> 262.7 mm, vias 5 -> 8
- net Net-(D3-A): track 6.42 -> 20.9 mm
- net Net-(D7-K): track 6.41 -> 18.7 mm
- net Net-(D15-K): track 7.11 -> 5.62 mm
- net Net-(D16-A): track 7.06 -> 5.60 mm
- net /PTSR: track 74.2 -> 72.9 mm
- net /PTTR: track 88.0 -> 86.8 mm, vias 4 -> 2

Commit message: Update PCB_Main
Routing:
- net VCC: track 262.7 -> 278.0 mm, vias 8 -> 5
- net /PTSR: track 72.9 -> 87.6 mm, vias 2 -> 4
- net GND: track 240.1 -> 246.8 mm
- net Net-(D7-K): track 18.7 -> 23.6 mm, vias 0 -> 2
- net +5V: track 210.2 -> 213.4 mm
- net Net-(D3-A): track 20.9 -> 19.0 mm

Commit message: Update PCB_Main
Routing:
- net +5V: track 213.4 -> 180.5 mm
- net Net-(D3-K): track 25.2 -> 43.8 mm
- net Net-(D4-K): track 35.5 -> 50.2 mm
- net VCC: track 278.0 -> 283.8 mm
- net Net-(D2-K): track 64.8 -> 64.1 mm
